File: pcb-files/Wave.kicad_sch (KiCad schematic)
At the start: 72 parts, among them IC1 NPM1300-QEAA-R, J1 USB4056-03-A_REVA2, J2 SJ-43516-SMT, J3 MEM2067-02-180-00-A_REVB, SW1 PTS815 SJM 250 SMTR LFS, SW2 PTS815 SJM 250 SMTR LFS, SW3 PTS815 SJM 250 SMTR LFS, U1 IM72D128V01XTMA1, U3 BT40F

Commit message: New Sch Doc with pin 17 for wifi module
Parts:
- added R130: 0, Resistor_SMD:R_0402_1005Metric, symbol Device:R
Connections:
- net 3.3V: now also R130.1
- net at U2.19 (OUT2P): now also C8.2
- new net: R130.2, U3.17 (wifi-pwr)
Changed lines of the file:
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@@
 	(wire
 		(pts
+			(xy 466.09 161.29) (xy 477.52 161.29)
+		)
+		(stroke
+			(width 0)
+			(type default)
+		)
+	)
+	(wire
+		(pts
 			(xy 393.7 231.14) (xy 414.02 231.14)
 		)
@@
 	(wire
 		(pts
+			(xy 452.12 161.29) (xy 458.47 161.29)
+		)
+		(stroke
+			(width 0)
+			(type default)
+		)
+	)
+	(wire
+		(pts
 			(xy 292.1 102.87) (xy 298.45 102.87)
 		)
@@
 	)
 	(label "3.3V"
+		(at 452.12 161.29 0)
+		(fields_autoplaced yes)
+		(effects
+			(font
+				(size 1.27 1.27)
+			)
+			(justify left bottom)
+		)
+	)
+	(label "3.3V"
 		(at 196.85 45.72 0)
 		(fields_autoplaced yes)
@@
 	)
 	(symbol
+		(lib_id "Device:R")
+		(at 462.28 161.29 90)
+		(unit 1)
+		(exclude_from_sim no)
+		(in_bom yes)
+		(on_board yes)
+		(dnp no)
+		(property "Reference" "R130"
+			(at 466.344 159.258 90)
+			(effects
+				(font
+					(size 1.27 1.27)
+				)
+			)
+		)
+		(property "Value" "0"
+			(at 458.978 159.512 90)
+			(effects
+				(font
+					(size 1.27 1.27)
+				)
+			)
+		)
+		(property "Footprint" "Resistor_SMD:R_0402_1005Metric"
+			(at 462.28 163.068 90)
+			(effects
+				(font
+					(size 1.27 1.27)
+				)
+				(hide yes)
+			)
+		)
+		(property "Datasheet" "~"
+			(at 462.28 161.29 0)
+			(effects
+				(font
+					(size 1.27 1.27)
+				)
+				(hide yes)
+			)
+		)
+		(property "Description" "Resistor"
+			(at 462.28 161.29 0)
+			(effects
+				(font
+					(size 1.27 1.27)
+				)
+				(hide yes)
+			)
+		)
+		(pin "2"
+		)
+		(pin "1"
+		)
+		(instances
+			(project "Wave"
+				(path "/4c47a525-f09f-4441-8def-34c50772c841"
+					(reference "R130")
+					(unit 1)
+				)
+			)
+		)
+	)
+	(symbol
 		(lib_id "Device:C")
 		(at 317.5 290.83 180)
@@
 		)
 		(instances
-			(project ""
+			(project "Wave"
 				(path "/4c47a525-f09f-4441-8def-34c50772c841"
 					(reference "R7")
@@
 		)
 		(instances
-			(project ""
+			(project "Wave"
 				(path "/4c47a525-f09f-4441-8def-34c50772c841"
 					(reference "U2")
@@
 		)
 		(instances
-			(project ""
+			(project "Wave"
 				(path "/4c47a525-f09f-4441-8def-34c50772c841"
 					(reference "R6")
@@
 		)
 		(instances
-			(project ""
+			(project "Wave"
 				(path "/4c47a525-f09f-4441-8def-34c50772c841"
 					(reference "1.2V1")
@@
 		(pin "A2"
 		)
+		(pin "17"
+		)
 		(instances

Commit message: Layout V1
First Layout of Wave v1
Parts:
- added J4: Conn_01x02, Connector_PinHeader_1.00mm:PinHeader_1x02_P1.00mm_Vertical, symbol PCM_4ms_Connector:Conn_01x02
- added PAD1: NTC, TestPoint:TestPoint_Pad_D2.0mm, symbol Connector:TestPoint
- added PAD2: VBAT, TestPoint:TestPoint_Pad_D2.0mm, symbol Connector:TestPoint
- added PAD3: GND, TestPoint:TestPoint_Pad_D2.0mm, symbol Connector:TestPoint
- added PAD4: GND, Battery:Battery_CR1225, symbol Connector:TestPoint
- IC1: footprint QFN50P500X500X90-33N -> WAVE:QFN50P500X500X90-33N
- U2: footprint Package_DFN_QFN:WAVE_CODEC -> WAVE:WAVE_CODEC
Connections:
- net PDM_DATA_MIC is gone; now on net PDM_DAT_MIC: U1.1 (DATA)
- net VBUS_5V is gone; now on net VBUSIN: R10.1
- net GND: now also PAD3.1
- net NTC_BAT: now also PAD1.1
- net SWCLK: now also J4.1 (Pin_1)
- net SWDIO: now also J4.2 (Pin_2)
- net VBAT: now also PAD2.1
- net OUT1P: now reaches C9.2, U2.20 (OUT1P)
- net DN2: now reaches D-1.1, U3.E5 (D-)
- net DP2: now reaches D+1.1, U3.E4 (D+)
- net IN1P: now reaches C6.2, U2.15 (IN1P)
- net OUT1M: now reaches U2.19 (OUT2M)
- net OUT1M: now also C8.2
Other:
- note added: "4/3/25"
- note added: "A"
- note added: "Battery"
- note added: "Program/Debug"
- note added: "WAVE"
- note added: "Wave Circuit Board"
